File: PCB/plus/nos_plus.kicad_pcb (KiCad board)
At the start: 2 copper layers, 576 x 92.1 mm, 159 parts, among them U1 PiPico_No_SWD, U2 ADG732BSUZ, U3 DC/DC

Commit message: Nos Pico+ PCB v1.0
Parts:
- added D63: MBR120VLSF, Diode_SMD:D_SOD-123, B.Cu at (39.0, 92.9)
- added SW1: SW_SPST, nos_plus:SW_Choc_V1V2_Cherry_MX_LED, F.Cu at (118.5, 159.6)
- added SW2: SW_SPST, nos_plus:SW_Choc_V1V2_Cherry_MX_LED, F.Cu at (138.5, 159.6)
- added SW3: SW_SPST, nos_plus:SW_Choc_V1V2_Cherry_MX_LED, F.Cu at (508.5, 159.6)
- added SW4: SW_SPST, nos_plus:SW_Choc_V1V2_Cherry_MX_LED, F.Cu at (488.5, 159.6)
- U1: footprint nos_main:RPi_Pico_SMD_Pins_No_SWD -> nos_plus:RPi_Pico_SMD_Pins_No_SWD
- U2: footprint nos_main:QFP50P900X900X120-49N -> nos_plus:QFP50P900X900X120-49N
- U3: footprint nos_main:DCDC_3to5 -> nos_plus:DCDC_3to5
- moved R1 135.0 mm to (52.2, 127.8)
- moved R2 134.9 mm to (52.2, 126.2)
- moved C15 118.8 mm to (320.3, 111.6)
- moved C14 112.1 mm to (300.3, 111.6)
- moved C13 101.5 mm to (280.3, 111.6)
- moved C30 99.2 mm to (52.2, 124.6), turned to 0 degrees
- moved C12 99.0 mm to (260.3, 111.6)
- moved C11 92.7 mm to (240.3, 111.6)
- moved U3 90.9 mm to (107.5, 109.6)
- moved C10 86.6 mm to (220.3, 111.6)
- moved C16 82.5 mm to (340.3, 111.6)
- moved C9 80.8 mm to (200.3, 111.6)
- moved C17 77.5 mm to (360.3, 111.6)
- moved C8 75.2 mm to (180.3, 111.6)
- moved C18 70.0 mm to (380.3, 111.6)
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Connections:
- U1 pad 14: unconnected-(U1-GPIO10-Pad14) -> Net-(SW4-B)
- U1 pad 15: unconnected-(U1-GPIO11-Pad15) -> Net-(SW3-B)
- U1 pad 16: unconnected-(U1-GPIO12-Pad16) -> Net-(SW2-B)
- U1 pad 17: unconnected-(U1-GPIO13-Pad17) -> Net-(SW1-B)
- U1 pad 40: VBUS -> unconnected-(U1-VBUS-Pad40)
- USB1 pad 11: VBUS -> Net-(D63-A)
- USB1 pad 2: VBUS -> Net-(D63-A)
Routing:
- net +5V: track 0.00 -> 1755.5 mm, vias 0 -> 4
- net Vref: track 0.00 -> 861.8 mm, vias 0 -> 3
- net Net-(SW3-B): track 0.00 -> 505.3 mm
- net Net-(SW4-B): track 0.00 -> 483.8 mm
- net Net-(D57-In): track 0.00 -> 303.7 mm, vias 0 -> 1
- net /WR: track 0.00 -> 280.7 mm, vias 0 -> 1
- net /A4: track 0.00 -> 279.4 mm, vias 0 -> 1
- net /CS: track 0.00 -> 279.1 mm, vias 0 -> 1
- net /A3: track 0.00 -> 278.8 mm, vias 0 -> 1
- net /A0: track 0.00 -> 277.3 mm, vias 0 -> 1
- net /A2: track 0.00 -> 276.8 mm, vias 0 -> 1
- net /A1: track 0.00 -> 276.5 mm, vias 0 -> 1
- net Net-(U2-D): track 0.00 -> 273.5 mm, vias 0 -> 3
- net /S28: track 0.00 -> 271.4 mm
- net /S1: track 0.00 -> 269.5 mm
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- added copper zone on B.Cu, net GND
- added copper zone on F.Cu, net GND

Commit message: Nos Pico + PCB v1.01 (footprint finetune)
Parts:
- D63: footprint Diode_SMD:D_SOD-123 -> nos_plus:D_SOD-123_LONG
- H1, H10, H11, H12, H13, H14, H15, H16, H17, H18, H19, H2, H20, H21, H22, H23, H24, H25, H26, H27, H28, H3, H4, H5, H6, H7, H8, H9: footprint Package_TO_SOT_SMD:SOT-23-3 -> nos_plus:SOT-23-FAT
- moved D63 0.14 mm to (39.2, 92.9)
Routing:
- net Net-(D1-In): track 22.8 -> 23.9 mm
Other:
- board text added: "Nos Pico+ v1.01"
- board text removed: "Nos Pico+ v1.0"

Commit message: PCB v1.2, remove unnecessary components
Parts:
- removed C30: 1nF, Capacitor_SMD:C_0603_1608Metric_Pad1.08x0.95mm_HandSolder
- removed JP1: SolderJumper_2_Open, Jumper:SolderJumper-2_P1.3mm_Open_RoundedPad1.0x1.5mm
- removed U3: DC/DC, nos_plus:DCDC_3to5
- added C61: 0.1uF, Capacitor_SMD:C_0603_1608Metric_Pad1.08x0.95mm_HandSolder, B.Cu at (110.7, 119.1)
- added C62: 0.1uF, Capacitor_SMD:C_0603_1608Metric_Pad1.08x0.95mm_HandSolder, B.Cu at (110.7, 126.2)
- added U6: LM4040DBZ-3, nos_plus:SOT-23-FAT, B.Cu at (42.1, 125.8)
- added U7: LP5907MFX-4.5, Package_TO_SOT_SMD:SOT-23-5, B.Cu at (112.5, 122.4)
- R2: value 10K -> 5.1K
Connections:
- U1 pad 35: unconnected-(U1-ADC_VREF-Pad35) -> Net-(U1-ADC_VREF)
Routing:
- net +3V3: track 76.6 -> 0.00 mm
- net Vref: track 861.8 -> 837.0 mm
- net +5V: track 1755.9 -> 1776.0 mm, vias 4 -> 5
- net GND: track 5.02 -> 23.4 mm, vias 190 -> 192
- net Net-(U1-ADC_VREF): track 0.00 -> 5.26 mm
Other:
- board text added: "Nos Pico+ v1.2"
- board text added: "github.com/whowechina"
- board text removed: "Nos Pico+ v1.01"
